Commit message: feat: update wq urdf

File: robotsky_lab/assets/robotsky_wq/urdf/robotsky_wq.urdf (robot description, URDF)
Before this commit: robot robotsky_wq, 17 links, 16 joints
Joints:
- joint LB_Hip_Joint: limit lower=-0.01 upper=3.14 effort=14 velocity=30 -> lower=-0.01 upper=3.14 effort=8 velocity=20
- joint LB_Knee_Joint: limit lower=-3.14 upper=0.01 effort=17 velocity=30 -> lower=-3.14 upper=0.01 effort=12 velocity=20
- joint LB_Roll_Joint: limit lower=-1.57 upper=0.5 effort=7 velocity=12 -> lower=-1.57 upper=0.5 effort=5 velocity=10
- joint LB_Wheel_Joint: limit lower=-300000000 upper=300000000 effort=7 velocity=12 -> effort=5 velocity=10; type revolute -> continuous
- joint LF_Hip_Joint: limit lower=-3.14 upper=0.01 effort=14 velocity=30 -> lower=-3.14 upper=0.01 effort=8 velocity=20
- joint LF_Knee_Joint: limit lower=-0.01 upper=3.14 effort=17 velocity=30 -> lower=-0.01 upper=3.14 effort=12 velocity=20
- joint LF_Roll_Joint: limit lower=-1.57 upper=0.5 effort=7 velocity=12 -> lower=-1.57 upper=0.5 effort=5 velocity=10
- joint LF_Wheel_Joint: limit lower=-300000000 upper=300000000 effort=7 velocity=12 -> effort=5 velocity=10; type revolute -> continuous
- joint RB_Hip_Joint: limit lower=-0.01 upper=3.14 effort=14 velocity=30 -> lower=-0.01 upper=3.14 effort=8 velocity=20
- joint RB_Knee_Joint: limit lower=-3.14 upper=0.01 effort=17 velocity=30 -> lower=-3.14 upper=0.01 effort=12 velocity=20
- joint RB_Roll_Joint: limit lower=-0.5 upper=1.57 effort=7 velocity=12 -> lower=-0.5 upper=1.57 effort=5 velocity=10
- joint RB_Wheel_Joint: limit lower=-300000000 upper=300000000 effort=7 velocity=12 -> effort=5 velocity=10; type revolute -> continuous
- joint RF_Hip_Joint: limit lower=-3.14 upper=0.01 effort=14 velocity=30 -> lower=-3.14 upper=0.01 effort=8 velocity=20
- joint RF_Knee_Joint: limit lower=-0.01 upper=3.14 effort=17 velocity=30 -> lower=-0.01 upper=3.14 effort=12 velocity=20
- joint RF_Roll_Joint: limit lower=-0.5 upper=1.57 effort=7 velocity=12 -> lower=-0.5 upper=1.57 effort=5 velocity=10
- joint RF_Wheel_Joint: limit lower=-300000000 upper=300000000 effort=7 velocity=12 -> effort=5 velocity=10; type revolute -> continuous

Commit message: feat: update urdf and robot model, update train config

File: robotsky_lab/assets/robotsky_wq/urdf/robotsky_wq.urdf (robot description, URDF)
Before this commit: robot robotsky_wq, 17 links, 16 joints
Links:
- link LB_Wheel_Link: geometry collision cylinder length=0.035 radius=0.075; visual cylinder length=0.035 radius=0.075
- link LF_Wheel_Link: geometry collision cylinder length=0.035 radius=0.075; visual cylinder length=0.035 radius=0.075
- link RB_Wheel_Link: geometry collision cylinder length=0.035 radius=0.075; visual cylinder length=0.035 radius=0.075
- link RF_Wheel_Link: geometry collision cylinder length=0.035 radius=0.075; visual cylinder length=0.035 radius=0.075

Commit message: feat: try to make a baseline version

File: robotsky_lab/assets/robotsky_wq/urdf/robotsky_wq.urdf (robot description, URDF)
Before this commit: robot robotsky_wq, 17 links, 16 joints
Links:
- link base_link: mass 10.2741064 -> 11.2741064
